Commit message: yubi: composite the Quest head into yubi_hands.urdf + declare the base head camera
The das-umi composite pattern: expand_yubi_xacro.py now grafts
quest3s_head (floating under quest_origin — an independently tracked
body) and quest3s_camera_optical (identity fixed joint; the measured
extrinsic rides the capture data, never the description). The three
yubi-* embodiments declare the QUEST3_HEAD 'base' camera on
quest3s_head, so a trainable yubi episode embodies the head view
exactly as das episodes do.

Co-Authored-By: Claude Fable 5 <noreply@anthropic.com>

File: assets/yubi_description/urdf/yubi_hands.urdf (robot description, URDF)
Before this commit: robot yubi_hands, 15 links, 14 joints
Links:
- added link quest3s_camera_optical
- added link quest3s_head
Joints:
- added joint quest3s_head_to_camera_optical: type fixed, parent quest3s_head, child quest3s_camera_optical, origin xyz=0 0 0 rpy=0 0 0
- added joint quest_origin_to_head: type floating, parent quest_origin, child quest3s_head, origin xyz=0 0 0 rpy=0 0 0
