Commit message: feat: update legacy urdf with existing physical gripper's urdf

File: assets/yubi_description/urdf/yubi_hands.urdf (robot description, URDF)
Before this commit: robot yubi_hands, 17 links, 16 joints
Links:
- removed link left_hand_cam_link
- removed link left_left_finger_link
- removed link left_left_finger_tip_link
- removed link left_right_finger_link
- removed link left_right_finger_tip_link
- removed link right_hand_cam_link
- removed link right_left_finger_link
- removed link right_left_finger_tip_link
- removed link right_right_finger_link
- removed link right_right_finger_tip_link
- added link left_base_link; collision mesh filename=package://yubi_description/meshes/left/link_housing.stl; visual mesh filename=package://yubi_description/meshes/left/link_housing.stl
- added link left_controller_link; collision mesh filename=package://yubi_description/meshes/left/link_controller.stl; visual mesh filename=package://yubi_description/meshes/left/link_controller.stl
- added link left_gripper_tip
- added link left_left_finger_grip
- added link left_left_nail; collision mesh filename=package://yubi_description/meshes/shared/link_left_nail.stl; visual mesh filename=package://yubi_description/meshes/shared/link_left_nail.stl
- added link left_link_connector_left; collision mesh filename=package://yubi_description/meshes/shared/link_connector.stl; visual mesh filename=package://yubi_description/meshes/shared/link_connector.stl
- added link left_link_connector_right; collision mesh filename=package://yubi_description/meshes/shared/link_connector.stl; visual mesh filename=package://yubi_description/meshes/shared/link_connector.stl
- added link left_link_left_finger; collision mesh filename=package://yubi_description/meshes/shared/link_left_finger.s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; visual mesh filename=package://yubi_description/meshes/shared/link_left_finger.s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
- added link left_link_right_finger; collision mesh filename=package://yubi_description/meshes/shared/link_right_finger.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; visual mesh filename=package://yubi_description/meshes/shared/link_right_finger.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
- added link left_right_finger_grip
- added link left_right_nail; collision mesh filename=package://yubi_description/meshes/shared/link_right_nail.stl; visual mesh filename=package://yubi_description/meshes/shared/link_right_nail.stl
- added link right_base_link; collision mesh filename=package://yubi_description/meshes/right/link_housing.stl; visual mesh filename=package://yubi_description/meshes/right/link_housing.stl
- added link right_controller_link; collision mesh filename=package://yubi_description/meshes/right/link_controller.stl; visual mesh filename=package://yubi_description/meshes/right/link_controller.stl
- added link right_gripper_tip
- added link right_left_finger_grip
- added link right_left_nail; collision mesh filename=package://yubi_description/meshes/shared/link_left_nail.stl; visual mesh filename=package://yubi_description/meshes/shared/link_left_nail.stl
- added link right_link_connector_left; collision mesh filename=package://yubi_description/meshes/shared/link_connector.stl; visual mesh filename=package://yubi_description/meshes/shared/link_connector.stl
- added link right_link_connector_right; collision mesh filename=package://yubi_description/meshes/shared/link_connector.stl; visual mesh filename=package://yubi_description/meshes/shared/link_connector.stl
- added link right_link_left_finger; collision mesh filename=package://yubi_description/meshes/shared/link_left_finger.s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; visual mesh filename=package://yubi_description/meshes/shared/link_left_finger.s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
- added link right_link_right_finger; collision mesh filename=package://yubi_description/meshes/shared/link_right_finger.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; visual mesh filename=package://yubi_description/meshes/shared/link_right_finger.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
- added link right_right_finger_grip
- added link right_right_nail; collision mesh filename=package://yubi_description/meshes/shared/link_right_nail.stl; visual mesh filename=package://yubi_description/meshes/shared/link_right_nail.stl
- link left_hand_root: geometry collision mesh filename=package://yubi_description/meshes/shared/link_base_link.stl; visual mesh filename=package://yubi_description/meshes/shared/link_base_link.stl
- link right_hand_root: geometry collision mesh filename=package://yubi_description/meshes/shared/link_base_link.stl; visual mesh filename=package://yubi_description/meshes/shared/link_base_link.stl
Joints:
- removed joint left_camera_joint
- removed joint left_camera_optical_joint
- removed joint left_left_finger_joint
- removed joint left_left_finger_tip_joint
- removed joint left_mount_joint
- removed joint left_right_finger_joint
- removed joint left_right_finger_tip_joint
- removed joint right_camera_joint
- removed joint right_camera_optical_joint
- removed joint right_left_finger_joint
- removed joint right_left_finger_tip_joint
- removed joint right_mount_joint
- removed joint right_right_finger_joint
- removed joint right_right_finger_tip_joint
- added joint left_camera_link_frame: type fixed, parent left_base_link, child left_hand_cam_optical, origin xyz=-0.00952825 -0 0.0362439 rpy=-1.74533 0 -1.5708
- added joint left_controller: type fixed, parent left_base_link, child left_controller_link, origin xyz=-0.063 0.016 0.0525 rpy=0 -0.7853981633974483 0.7853981633974483
- added joint left_controller_tracking_frame: type fixed, parent left_controller_link, child quest_left_controller, origin xyz=0 0 0 rpy=0 0 -1.5707963267948966
- added joint left_gripper_tip_frame: type fixed, parent left_base_link, child left_gripper_tip, origin xyz=0.0875496611 0 -0.00605006867 rpy=0 0 0
- added joint left_left_connector: type revolute, parent left_base_link, child left_link_connector_left, origin xyz=-0.016 0.0550024899162 -0.00380014595406 rpy=-0.00000000537222922 -0.000000170962516 -0.0157353974, axis 0 0 1, limit lower=-3.141592653589793 upper=3.141592653589793 effort=10 velocity=10, mimic joint=left_left_finger multiplier=1 offset=0
- added joint left_left_finger: type revolute, parent left_base_link, child left_link_left_finger, origin xyz=-0.0159999253 0.01500011285 0.01200007484 rpy=0 0 -0.0349065974, axis 0 0 1, limit lower=0 upper=0.785398 effort=10 velocity=10
- added joint left_left_finger_grip_frame: type fixed, parent left_link_left_finger, child left_left_finger_grip, origin xyz=0.0647084 0.00546061 -0.01775 rpy=-1e-12 0 -0
- added joint left_left_nail: type revolute, parent left_link_connector_left, child left_left_nail, origin xyz=0.0670678187713 -0.00845642917701 -0.00049967119931 rpy=-1.33006886754e-12 8.45202241528e-11 0, axis 0 0 1, limit lower=-3.141592653589793 upper=3.141592653589793 effort=10 velocity=10, mimic joint=left_left_finger multiplier=-1 offset=0
- added joint left_right_connector: type revolute, parent left_base_link, child left_link_connector_right, origin xyz=-0.016 -0.0549975100834 -0.00379985405918 rpy=-0.00000000382026972 0.000000093109623 0.0245406753, axis 0 0 1, limit lower=-3.141592653589793 upper=3.141592653589793 effort=10 velocity=10, mimic joint=left_left_finger multiplier=-1 offset=0
- added joint left_right_finger: type revolute, parent left_base_link, child left_link_right_finger, origin xyz=-0.01600004037 -0.01500001935 0.01200007658 rpy=0 0 0.0349065753, axis 0 0 1, limit lower=-0.785398 upper=0 effort=10 velocity=10, mimic joint=left_left_finger multiplier=-1 offset=0
- added joint left_right_finger_grip_frame: type fixed, parent left_link_right_finger, child left_right_finger_grip, origin xyz=0.0646994 -0.00556635 -0.01775 rpy=1e-12 0 0
- added joint left_right_nail: type revolute, parent left_link_connector_right, child left_right_nail, origin xyz=0.0671849851405 0.00763956789707 0.00209999225656 rpy=-2.30027455417e-12 -9.37143695978e-11 0, axis 0 0 1, limit lower=-3.141592653589793 upper=3.141592653589793 effort=10 velocity=10, mimic joint=left_left_finger multiplier=1 offset=0
- added joint left_world_to_base_link: type fixed, parent left_hand_root, child left_base_link, origin xyz=0.014368 0 0.05331 rpy=-0 0.174533 -0
- added joint right_camera_link_frame: type fixed, parent right_base_link, child right_hand_cam_optical, origin xyz=-0.00952825 -0 0.0362439 rpy=-1.74533 0 -1.5708
- added joint right_controller: type fixed, parent right_base_link, child right_controller_link, origin xyz=-0.063 -0.016 0.0525 rpy=0 -0.7853981633974483 -0.7853981633974483
- added joint right_controller_tracking_frame: type fixed, parent right_controller_link, child quest_right_controller, origin xyz=0 0 0 rpy=0 0 -1.5707963267948966
- added joint right_gripper_tip_frame: type fixed, parent right_base_link, child right_gripper_tip, origin xyz=0.0875496611 0 -0.00605006867 rpy=0 0 0
- added joint right_left_connector: type revolute, parent right_base_link, child right_link_connector_left, origin xyz=-0.016 0.0550024899162 -0.00380014595406 rpy=-0.00000000537222922 -0.000000170962516 -0.0157353974, axis 0 0 1, limit lower=-3.141592653589793 upper=3.141592653589793 effort=10 velocity=10, mimic joint=right_left_finger multiplier=1 offset=0
- added joint right_left_finger: type revolute, parent right_base_link, child right_link_left_finger, origin xyz=-0.0159999253 0.01500011285 0.01200007484 rpy=0 0 -0.0349065974, axis 0 0 1, limit lower=0 upper=0.785398 effort=10 velocity=10
- added joint right_left_finger_grip_frame: type fixed, parent right_link_left_finger, child right_left_finger_grip, origin xyz=0.0647084 0.00546061 -0.01775 rpy=-1e-12 0 -0
- added joint right_left_nail: type revolute, parent right_link_connector_left, child right_left_nail, origin xyz=0.0670678187713 -0.00845642917701 -0.00049967119931 rpy=-1.33006886754e-12 8.45202241528e-11 0, axis 0 0 1, limit lower=-3.141592653589793 upper=3.141592653589793 effort=10 velocity=10, mimic joint=right_left_finger multiplier=-1 offset=0
- added joint right_right_connector: type revolute, parent right_base_link, child right_link_connector_right, origin xyz=-0.016 -0.0549975100834 -0.00379985405918 rpy=-0.00000000382026972 0.000000093109623 0.0245406753, axis 0 0 1, limit lower=-3.141592653589793 upper=3.141592653589793 effort=10 velocity=10, mimic joint=right_left_finger multiplier=-1 offset=0
- added joint right_right_finger: type revolute, parent right_base_link, child right_link_right_finger, origin xyz=-0.01600004037 -0.01500001935 0.01200007658 rpy=0 0 0.0349065753, axis 0 0 1, limit lower=-0.785398 upper=0 effort=10 velocity=10, mimic joint=right_left_finger multiplier=-1 offset=0
- added joint right_right_finger_grip_frame: type fixed, parent right_link_right_finger, child right_right_finger_grip, origin xyz=0.0646994 -0.00556635 -0.01775 rpy=1e-12 0 0
- added joint right_right_nail: type revolute, parent right_link_connector_right, child right_right_nail, origin xyz=0.0671849851405 0.00763956789707 0.00209999225656 rpy=-2.30027455417e-12 -9.37143695978e-11 0, axis 0 0 1, limit lower=-3.141592653589793 upper=3.141592653589793 effort=10 velocity=10, mimic joint=right_left_finger multiplier=1 offset=0
- added joint right_world_to_base_link: type fixed, parent right_hand_root, child right_base_link, origin xyz=0.014368 0 0.05331 rpy=-0 0.174533 -0
