Commit message: Fix composite embodiment descriptions

File: assets/das_gripper_with_vr/urdf/DAS_UMI_V4.urdf (robot description, URDF)
Before this commit: robot das_umi_v4, 44 links, 43 joints
Joints:
- joint head_to_left_rig: origin xyz=0 0 0 rpy=0 0 0 -> xyz=0 0.16 0 rpy=0 0 0; type fixed -> floating
- joint head_to_right_rig: origin xyz=0 0 0 rpy=0 0 0 -> xyz=0 -0.16 0 rpy=0 0 0; type fixed -> floating

File: assets/official/yor/yor.urdf (robot description, URDF)
Before this commit: robot cone-e, 32 links, 31 joints
Links:
- added link yor_origin
Joints:
- added joint yor_origin_to_base: type fixed, parent yor_origin, child base, origin xyz=0.00000000 0.00000000 0.10477502 rpy=0 1.57 0

File: assets/yubi_description/urdf/yubi_hands.urdf (robot description, URDF)
Before this commit: robot yubi_hands, 17 links, 16 joints
Joints:
- joint quest_origin_to_left: origin xyz=0 0 0 rpy=0 0 0 -> xyz=0 0.16 0 rpy=0 0 0
- joint quest_origin_to_right: origin xyz=0 0 0 rpy=0 0 0 -> xyz=0 -0.16 0 rpy=0 0 0

Commit message: Model Quest stereo capture rigs

File: assets/das_gripper_with_vr/urdf/DAS_UMI_V4.urdf (robot description, URDF)
Before this commit: robot das_umi_v4, 44 links, 43 joints
Links:
- added link quest3s_right_camera_optical
Joints:
- removed joint quest3s_head_to_camera_optical
- added joint quest3s_head_to_left_camera_optical: type fixed, parent quest3s_head, child quest3s_camera_optical, origin xyz=0 0 0 rpy=0 0 0
- added joint quest3s_head_to_right_camera_optical: type fixed, parent quest3s_head, child quest3s_right_camera_optical, origin xyz=0 0 0 rpy=0 0 0

File: assets/quest_ego/urdf/quest_ego.urdf (robot description, URDF)
Before this commit: robot quest_ego, 2 links, 1 joints
Links:
- added link quest3s_right_camera_optical
- link quest3s_head: geometry visual mesh filename=package://sx-embodiments/quest_ego/meshes/quest3mesh.obj scale=1 1 1
Joints:
- added joint quest3s_head_to_right_camera_optical: type fixed, parent quest3s_head, child quest3s_right_camera_optical, origin xyz=0 0 0 rpy=0 0 0

File: assets/yubi_description/urdf/yubi_hands.urdf (robot description, URDF)
Before this commit: robot yubi_hands, 17 links, 16 joints
Links:
- added link quest3s_right_camera_optical
Joints:
- removed joint quest3s_head_to_camera_optical
- added joint quest3s_head_to_left_camera_optical: type fixed, parent quest3s_head, child quest3s_camera_optical, origin xyz=0 0 0 rpy=0 0 0
- added joint quest3s_head_to_right_camera_optical: type fixed, parent quest3s_head, child quest3s_right_camera_optical, origin xyz=0 0 0 rpy=0 0 0

Commit message: Add Quest headset surfaces to capture rigs

File: assets/das_gripper_with_vr/urdf/DAS_UMI_V4.urdf (robot description, URDF)
Before this commit: robot das_umi_v4, 45 links, 44 joints
Links:
- link quest3s_head: geometry visual mesh filename=package://sx-embodiments/quest_ego/meshes/quest3mesh.obj

File: assets/yubi_description/urdf/yubi_hands.urdf (robot description, URDF)
Before this commit: robot yubi_hands, 18 links, 17 joints
Links:
- link quest3s_head: geometry visual mesh filename=package://sx-embodiments/quest_ego/meshes/quest3mesh.obj

Commit message: fix: make embodiment camera facts authoritative

File: assets/das_gripper_with_vr/urdf/DAS_UMI_V4.urdf (robot description, URDF)
Before this commit: robot das_umi_v4, 45 links, 44 joints
Joints:
- joint quest3s_head_to_left_camera_optical: origin xyz=0 0 0 rpy=0 0 0 -> xyz=-0.032 0.075 -0.011 rpy=-1.5707963267948966 0 0
- joint quest3s_head_to_right_camera_optical: origin xyz=0 0 0 rpy=0 0 0 -> xyz=0.032 0.075 -0.011 rpy=-1.5707963267948966 0 0

File: assets/quest_ego/urdf/quest_ego.urdf (robot description, URDF)
Before this commit: robot quest_ego, 3 links, 2 joints
Joints:
- joint quest3s_head_to_camera_optical: origin xyz=0 0 0 rpy=0 0 0 -> xyz=-0.032 0.075 -0.011 rpy=-1.5707963267948966 0 0
- joint quest3s_head_to_right_camera_optical: origin xyz=0 0 0 rpy=0 0 0 -> xyz=0.032 0.075 -0.011 rpy=-1.5707963267948966 0 0

File: assets/yubi_description/urdf/yubi_hands.urdf (robot description, URDF)
Before this commit: robot yubi_hands, 18 links, 17 joints
Links:
- removed link quest3s_camera_optical
- removed link quest3s_head
- removed link quest3s_right_camera_optical
Joints:
- removed joint quest3s_head_to_left_camera_optical
- removed joint quest3s_head_to_right_camera_optical
- removed joint quest_origin_to_head

Commit message: chore: tightening for yubi pods

File: assets/das_gripper_with_vr/urdf/DAS_UMI_V4.urdf (robot description, URDF)
Before this commit: robot das_umi_v4, 45 links, 44 joints
Links:
- removed link quest3s_camera_optical
- added link quest3s_left_camera_optical
Joints:
- joint quest3s_head_to_left_camera_optical: child quest3s_camera_optical -> quest3s_left_camera_optical

File: assets/quest_ego/urdf/quest_ego.urdf (robot description, URDF)
Before this commit: robot quest_ego, 3 links, 2 joints
Links:
- removed link quest3s_camera_optical
- added link quest3s_left_camera_optical
Joints:
- removed joint quest3s_head_to_camera_optical
- added joint quest3s_head_to_left_camera_optical: type fixed, parent quest3s_head, child quest3s_left_camera_optical, origin xyz=-0.032 0.075 -0.011 rpy=-1.5707963267948966 0 0

File: assets/yubi_description/urdf/yubi_hand.urdf.xacro (robot description, xacro)
@@ -47,4 +47,13 @@
       </collision>
     </link>
+    <!-- The upstream camera mount is already expressed in the camera's RDF
+         optical basis. Give that basis an explicit, symmetric frame name so
+         recordings and the description package name the same frame. -->
+    <joint name="${hand_prefix}_camera_optical_joint" type="fixed">
+      <origin xyz="0 0 0" rpy="0 0 0"/>
+      <parent link="${hand_prefix}_hand_cam_link"/>
+      <child link="${hand_prefix}_hand_cam_optical"/>
+    </joint>
+    <link name="${hand_prefix}_hand_cam_optical" data-frame-convention="camera_optical"/>
     <!-- Primary finger (driven directly by encoder) -->
     <joint name="${hand_prefix}_right_finger_joint" type="revolute">

File: assets/yubi_description/urdf/yubi_hands.urdf (robot description, URDF)
Before this commit: robot yubi_hands, 15 links, 14 joints
Links:
- added link left_hand_cam_optical
- added link right_hand_cam_optical
Joints:
- added joint left_camera_optical_joint: type fixed, parent left_hand_cam_link, child left_hand_cam_optical, origin xyz=0 0 0 rpy=0 0 0
- added joint right_camera_optical_joint: type fixed, parent right_hand_cam_link, child right_hand_cam_optical, origin xyz=0 0 0 rpy=0 0 0
