Commit message: Collide the RWH against convex parts, not its 1.4M-triangle visual meshes
The SolidWorks export pointed every <collision> at the full-detail visual mesh:
1,408,259 triangles across 58 links, base_link alone at 95,859. Upstream now derives
a CoACD convex decomposition per link and publishes urdf/sentient_rwh.urdf, and this
vendors it:

    collision 1,408,259 -> 80,202 triangles (18x cheaper), 1,366 convex parts

Kinematics and inertials are unchanged -- joint types, origins, axes, parents and
link masses all compare equal to the raw export -- so the 24-channel layout, the
footprint, and the embodiment's shape are untouched. Only the id moves, because
provenance and the URDF digest are part of the content hash.

The vendored description is now upstream's file byte-for-byte: the `v3` ->
`sentient_rwh` package rename moved into the generator, so there is no vendoring
patch left on this side to describe or drift.

test_urdf_parity gains a check that collision references resolve to convex parts and
never to a visual mesh. Re-vendoring the raw export would otherwise silently undo
this with identical kinematics, which nothing else would catch.

No regenerate-and-compare test, unlike yubi's composed URDF: CoACD's MCTS ignores its
seed, so regeneration is not byte-reproducible and such a test would flake. The
artifacts are pinned by digest instead.

Co-Authored-By: Claude Opus 5 <noreply@anthropic.com>

File: assets/sentient_rwh/urdf/sentient_rwh.urdf (robot description, URDF)
Before this commit: robot sentient_rwh, 58 links, 57 joints
Links:
- link Arm_link1: geometry collision mesh filename=package://sentient_rwh/meshes/collision/Arm_link1/Arm_link1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; collision mesh filename=package://sentient_rwh/meshes/collision/Arm_link1/Arm_link1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
- link Arm_link2: geometry collision mesh filename=package://sentient_rwh/meshes/collision/Arm_link2/Arm_link2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; collision mesh filename=package://sentient_rwh/meshes/collision/Arm_link2/Arm_link2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
- link Arm_link3: geometry collision mesh filename=package://sentient_rwh/meshes/collision/Arm_link3/Arm_link3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; collision mesh filename=package://sentient_rwh/meshes/collision/Arm_link3/Arm_link3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
- link Arm_link4: geometry collision mesh filename=package://sentient_rwh/meshes/collision/Arm_link4/Arm_link4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; collision mesh filename=package://sentient_rwh/meshes/collision/Arm_link4/Arm_link4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
- link Arm_link5_torso: geometry collision mesh filename=package://sentient_rwh/meshes/collision/Arm_link5_torso/Arm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; collision mesh filename=package://sentient_rwh/meshes/collision/Arm_link5_torso/Arm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
- link FL_tyre: geometry collision mesh filename=package://sentient_rwh/meshes/collision/FL_tyre/FL_tyre_000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; collision mesh filename=package://sentient_rwh/meshes/collision/FL_tyre/FL_tyre_001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
- link FR_tyre: geometry collision mesh filename=package://sentient_rwh/meshes/collision/FR_tyre/FR_tyre_000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; collision mesh filename=package://sentient_rwh/meshes/collision/FR_tyre/FR_tyre_001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
- link LA_1: geometry collision mesh filename=package://sentient_rwh/meshes/collision/LA_1/LA_1_000.stl; collision mesh filename=package://sentient_rwh/meshes/collision/LA_1/LA_1_001.stl
- link LA_2: geometry collision mesh filename=package://sentient_rwh/meshes/collision/LA_2/LA_2_000.stl; collision mesh filename=package://sentient_rwh/meshes/collision/LA_2/LA_2_001.stl
- link LA_3: geometry collision mesh filename=package://sentient_rwh/meshes/collision/LA_3/LA_3_000.stl; collision mesh filename=package://sentient_rwh/meshes/collision/LA_3/LA_3_001.stl
- link LA_4: geometry collision mesh filename=package://sentient_rwh/meshes/collision/LA_4/LA_4_000.stl; collision mesh filename=package://sentient_rwh/meshes/collision/LA_4/LA_4_001.stl
- link LA_5: geometry collision mesh filename=package://sentient_rwh/meshes/collision/LA_5/LA_5_000.stl; collision mesh filename=package://sentient_rwh/meshes/collision/LA_5/LA_5_001.stl
- link LA_6: geometry collision mesh filename=package://sentient_rwh/meshes/collision/LA_6/LA_6_000.stl; collision mesh filename=package://sentient_rwh/meshes/collision/LA_6/LA_6_001.stl
- link LA_7: geometry collision mesh filename=package://sentient_rwh/meshes/collision/LA_7/LA_7_000.stl; collision mesh filename=package://sentient_rwh/meshes/collision/LA_7/LA_7_001.stl
- link LA_8_wrist: geometry collision mesh filename=package://sentient_rwh/meshes/collision/LA_8_wrist/LA_8_wri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; collision mesh filename=package://sentient_rwh/meshes/collision/LA_8_wrist/LA_8_wri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
- link LA_Finger1_1: geometry collision mesh filename=package://sentient_rwh/meshes/collision/LA_Finger1_1/LA_Fin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; collision mesh filename=package://sentient_rwh/meshes/collision/LA_Finger1_1/LA_Fin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
- link LA_Finger1_2: geometry collision mesh filename=package://sentient_rwh/meshes/collision/LA_Finger1_2/LA_Fin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; collision mesh filename=package://sentient_rwh/meshes/collision/LA_Finger1_2/LA_Fin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
- link LA_Finger1_3: geometry collision mesh filename=package://sentient_rwh/meshes/collision/LA_Finger1_3/LA_Fin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; collision mesh filename=package://sentient_rwh/meshes/collision/LA_Finger1_3/LA_Fin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
- link LA_Finger1_4: geometry collision mesh filename=package://sentient_rwh/meshes/collision/LA_Finger1_4/LA_Fin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; collision mesh filename=package://sentient_rwh/meshes/collision/LA_Finger1_4/LA_Fin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
- link LA_Finger2_1: geometry collision mesh filename=package://sentient_rwh/meshes/collision/LA_Finger2_1/LA_Fin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; collision mesh filename=package://sentient_rwh/meshes/collision/LA_Finger2_1/LA_Fin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
- link LA_Finger2_2: geometry collision mesh filename=package://sentient_rwh/meshes/collision/LA_Finger2_2/LA_Fin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; collision mesh filename=package://sentient_rwh/meshes/collision/LA_Finger2_2/LA_Fin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
- link LA_Finger2_3: geometry collision mesh filename=package://sentient_rwh/meshes/collision/LA_Finger2_3/LA_Fin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; collision mesh filename=package://sentient_rwh/meshes/collision/LA_Finger2_3/LA_Fin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
- link LA_Finger2_4: geometry collision mesh filename=package://sentient_rwh/meshes/collision/LA_Finger2_4/LA_Fin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; collision mesh filename=package://sentient_rwh/meshes/collision/LA_Finger2_4/LA_Fin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
- link LA_Finger3_1: geometry collision mesh filename=package://sentient_rwh/meshes/collision/LA_Finger3_1/LA_Fin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; collision mesh filename=package://sentient_rwh/meshes/collision/LA_Finger3_1/LA_Fin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
- link LA_Finger3_2: geometry collision mesh filename=package://sentient_rwh/meshes/collision/LA_Finger3_2/LA_Fin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; collision mesh filename=package://sentient_rwh/meshes/collision/LA_Finger3_2/LA_Fin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
- link LA_Finger3_3: geometry collision mesh filename=package://sentient_rwh/meshes/collision/LA_Finger3_3/LA_Fin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; collision mesh filename=package://sentient_rwh/meshes/collision/LA_Finger3_3/LA_Fin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
- link LA_Finger3_4: geometry collision mesh filename=package://sentient_rwh/meshes/collision/LA_Finger3_4/LA_Fin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; collision mesh filename=package://sentient_rwh/meshes/collision/LA_Finger3_4/LA_Fin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
- link LA_Thumb_1: geometry collision mesh filename=package://sentient_rwh/meshes/collision/LA_Thumb_1/LA_Thumb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; collision mesh filename=package://sentient_rwh/meshes/collision/LA_Thumb_1/LA_Thumb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
- link LA_Thumb_2: geometry collision mesh filename=package://sentient_rwh/meshes/collision/LA_Thumb_2/LA_Thumb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; collision mesh filename=package://sentient_rwh/meshes/collision/LA_Thumb_2/LA_Thumb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
- link LA_Thumb_3: geometry collision mesh filename=package://sentient_rwh/meshes/collision/LA_Thumb_3/LA_Thumb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; collision mesh filename=package://sentient_rwh/meshes/collision/LA_Thumb_3/LA_Thumb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
- link LA_Thumb_4: geometry collision mesh filename=package://sentient_rwh/meshes/collision/LA_Thumb_4/LA_Thumb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; collision mesh filename=package://sentient_rwh/meshes/collision/LA_Thumb_4/LA_Thumb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
- link RA_1: geometry collision mesh filename=package://sentient_rwh/meshes/collision/RA_1/RA_1_000.stl; collision mesh filename=package://sentient_rwh/meshes/collision/RA_1/RA_1_001.stl
- link RA_2: geometry collision mesh filename=package://sentient_rwh/meshes/collision/RA_2/RA_2_000.stl; collision mesh filename=package://sentient_rwh/meshes/collision/RA_2/RA_2_001.stl
- link RA_3: geometry collision mesh filename=package://sentient_rwh/meshes/collision/RA_3/RA_3_000.stl; collision mesh filename=package://sentient_rwh/meshes/collision/RA_3/RA_3_001.stl
- link RA_4: geometry collision mesh filename=package://sentient_rwh/meshes/collision/RA_4/RA_4_000.stl; collision mesh filename=package://sentient_rwh/meshes/collision/RA_4/RA_4_001.stl
- link RA_5: geometry collision mesh filename=package://sentient_rwh/meshes/collision/RA_5/RA_5_000.stl; collision mesh filename=package://sentient_rwh/meshes/collision/RA_5/RA_5_001.stl
- link RA_6: geometry collision mesh filename=package://sentient_rwh/meshes/collision/RA_6/RA_6_000.stl; collision mesh filename=package://sentient_rwh/meshes/collision/RA_6/RA_6_001.stl
- link RA_7: geometry collision mesh filename=package://sentient_rwh/meshes/collision/RA_7/RA_7_000.stl; collision mesh filename=package://sentient_rwh/meshes/collision/RA_7/RA_7_001.stl
- link RA_8: geometry collision mesh filename=package://sentient_rwh/meshes/collision/RA_8/RA_8_000.stl; collision mesh filename=package://sentient_rwh/meshes/collision/RA_8/RA_8_001.stl
- link RA_Finger1_1: geometry collision mesh filename=package://sentient_rwh/meshes/collision/RA_Finger1_1/RA_Fin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; collision mesh filename=package://sentient_rwh/meshes/collision/RA_Finger1_1/RA_Fin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
- link RA_Finger1_2: geometry collision mesh filename=package://sentient_rwh/meshes/collision/RA_Finger1_2/RA_Fin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; collision mesh filename=package://sentient_rwh/meshes/collision/RA_Finger1_2/RA_Fin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
- link RA_Finger1_3: geometry collision mesh filename=package://sentient_rwh/meshes/collision/RA_Finger1_3/RA_Fin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; collision mesh filename=package://sentient_rwh/meshes/collision/RA_Finger1_3/RA_Fin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
- link RA_Finger1_4: geometry collision mesh filename=package://sentient_rwh/meshes/collision/RA_Finger1_4/RA_Fin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; collision mesh filename=package://sentient_rwh/meshes/collision/RA_Finger1_4/RA_Fin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
- link RA_Finger2_1: geometry collision mesh filename=package://sentient_rwh/meshes/collision/RA_Finger2_1/RA_Fin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; collision mesh filename=package://sentient_rwh/meshes/collision/RA_Finger2_1/RA_Fin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
- link RA_Finger2_2: geometry collision mesh filename=package://sentient_rwh/meshes/collision/RA_Finger2_2/RA_Fin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; collision mesh filename=package://sentient_rwh/meshes/collision/RA_Finger2_2/RA_Fin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
- link RA_Finger2_3: geometry collision mesh filename=package://sentient_rwh/meshes/collision/RA_Finger2_3/RA_Fin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; collision mesh filename=package://sentient_rwh/meshes/collision/RA_Finger2_3/RA_Fin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
- link RA_Finger2_4: geometry collision mesh filename=package://sentient_rwh/meshes/collision/RA_Finger2_4/RA_Fin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; collision mesh filename=package://sentient_rwh/meshes/collision/RA_Finger2_4/RA_Fin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
- link RA_Finger3_1: geometry collision mesh filename=package://sentient_rwh/meshes/collision/RA_Finger3_1/RA_Fin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; collision mesh filename=package://sentient_rwh/meshes/collision/RA_Finger3_1/RA_Fin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
- link RA_Finger3_2: geometry collision mesh filename=package://sentient_rwh/meshes/collision/RA_Finger3_2/RA_Fin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; collision mesh filename=package://sentient_rwh/meshes/collision/RA_Finger3_2/RA_Fin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
- link RA_Finger3_3: geometry collision mesh filename=package://sentient_rwh/meshes/collision/RA_Finger3_3/RA_Fin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; collision mesh filename=package://sentient_rwh/meshes/collision/RA_Finger3_3/RA_Fin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
- link RA_Finger3_4: geometry collision mesh filename=package://sentient_rwh/meshes/collision/RA_Finger3_4/RA_Fin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; collision mesh filename=package://sentient_rwh/meshes/collision/RA_Finger3_4/RA_Fin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
- link RA_THUMB_1: geometry collision mesh filename=package://sentient_rwh/meshes/collision/RA_THUMB_1/RA_THUMB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; collision mesh filename=package://sentient_rwh/meshes/collision/RA_THUMB_1/RA_THUMB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
- link RA_THUMB_2: geometry collision mesh filename=package://sentient_rwh/meshes/collision/RA_THUMB_2/RA_THUMB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; collision mesh filename=package://sentient_rwh/meshes/collision/RA_THUMB_2/RA_THUMB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
- link RA_THUMB_3: geometry collision mesh filename=package://sentient_rwh/meshes/collision/RA_THUMB_3/RA_THUMB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; collision mesh filename=package://sentient_rwh/meshes/collision/RA_THUMB_3/RA_THUMB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
- link RA_THUMB_4: geometry collision mesh filename=package://sentient_rwh/meshes/collision/RA_THUMB_4/RA_THUMB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; collision mesh filename=package://sentient_rwh/meshes/collision/RA_THUMB_4/RA_THUMB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
- link RL_tyre: geometry collision mesh filename=package://sentient_rwh/meshes/collision/RL_tyre/RL_tyre_000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; collision mesh filename=package://sentient_rwh/meshes/collision/RL_tyre/RL_tyre_001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
- link RR_tyre: geometry collision mesh filename=package://sentient_rwh/meshes/collision/RR_tyre/RR_tyre_000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; collision mesh filename=package://sentient_rwh/meshes/collision/RR_tyre/RR_tyre_001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
- link base_link: geometry collision mesh filename=package://sentient_rwh/meshes/collision/base_link/base_link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; collision mesh filename=package://sentient_rwh/meshes/collision/base_link/base_link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
