Commit message: Compose embodiments and package simulation assets and previews

File: assets/official/aloha/aloha.urdf (robot description, URDF)
Before this commit: robot aloha, 29 links, 28 joints
Links:
- link left/gripper_bar_link: geometry collision mesh filename=package://sx-embodiments/official/aloha/meshes/vx300s_9_gri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 scale=0.001 0.001 0.001; visual mesh filename=package://sx-embodiments/official/aloha/meshes/vx300s_9_gri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 scale=0.001 0.001 0.001
- link left/gripper_prop_link: geometry collision mesh filename=package://sx-embodiments/official/aloha/meshes/vx300s_8_gri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 scale=0.001 0.001 0.001; visual mesh filename=package://sx-embodiments/official/aloha/meshes/vx300s_8_gri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 scale=0.001 0.001 0.001
- link left/left_finger_link: geometry collision mesh filename=package://sx-embodiments/official/aloha/meshes/vx300s_10_gr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 scale=0.001 0.001 0.001; visual mesh filename=package://sx-embodiments/official/aloha/meshes/vx300s_10_gr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 scale=0.001 0.001 0.001
- link left/right_finger_link: geometry collision mesh filename=package://sx-embodiments/official/aloha/meshes/vx300s_10_gr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 scale=0.001 0.001 0.001; visual mesh filename=package://sx-embodiments/official/aloha/meshes/vx300s_10_gr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 scale=0.001 0.001 0.001
- link right/gripper_bar_link: geometry collision mesh filename=package://sx-embodiments/official/aloha/meshes/vx300s_9_gri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 scale=0.001 0.001 0.001; visual mesh filename=package://sx-embodiments/official/aloha/meshes/vx300s_9_gri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 scale=0.001 0.001 0.001
- link right/gripper_prop_link: geometry collision mesh filename=package://sx-embodiments/official/aloha/meshes/vx300s_8_gri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 scale=0.001 0.001 0.001; visual mesh filename=package://sx-embodiments/official/aloha/meshes/vx300s_8_gri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 scale=0.001 0.001 0.001
- link right/left_finger_link: geometry collision mesh filename=package://sx-embodiments/official/aloha/meshes/vx300s_10_gr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 scale=0.001 0.001 0.001; visual mesh filename=package://sx-embodiments/official/aloha/meshes/vx300s_10_gr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 scale=0.001 0.001 0.001
- link right/right_finger_link: geometry collision mesh filename=package://sx-embodiments/official/aloha/meshes/vx300s_10_gr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 scale=0.001 0.001 0.001; visual mesh filename=package://sx-embodiments/official/aloha/meshes/vx300s_10_gr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 scale=0.001 0.001 0.001
