Commit message: Add independent Yubi controller-holder CAD reference frames

File: assets/yubi_description/source/yubi_left_gripper.urdf (robot description, URDF)
Before this commit: robot left_gripper_v2_final, 13 links, 12 joints
Links:
- added link controller_holder
Joints:
- added joint controller_holder_frame: type fixed, parent base_link, child controller_holder, origin xyz=-0.038000038116582681 0.0074997656908985322 0.013999894092481618 rpy=-4.0314486803392608e-08 8.9708139361377448e-07 4.607911508865901e-07

File: assets/yubi_description/source/yubi_right_gripper.urdf (robot description, URDF)
Before this commit: robot right_gripper_corrected_fixed, 13 links, 12 joints
Links:
- added link controller_holder
Joints:
- added joint controller_holder_frame: type fixed, parent base_link, child controller_holder, origin xyz=-0.037999977854557943 -0.0075000000003000063 0.01399997281189156 rpy=4.5777735220020544e-16 -7.4800567295696396e-08 8.0718499414803019e-17

File: assets/yubi_description/urdf/yubi_hands.urdf (robot description, URDF)
Before this commit: robot yubi_hands, 29 links, 28 joints
Links:
- added link left_controller_holder
- added link right_controller_holder
Joints:
- added joint left_controller_holder_frame: type fixed, parent left_base_link, child left_controller_holder, origin xyz=-0.038000038116582681 0.0074997656908985322 0.013999894092481618 rpy=-4.0314486803392608e-08 8.9708139361377448e-07 4.607911508865901e-07
- added joint right_controller_holder_frame: type fixed, parent right_base_link, child right_controller_holder, origin xyz=-0.037999977854557943 -0.0075000000003000063 0.01399997281189156 rpy=4.5777735220020544e-16 -7.4800567295696396e-08 8.0718499414803019e-17

Commit message: Separate independent Yubi holder-frame changes from Piper support

File: assets/yubi_description/source/yubi_left_gripper.urdf (robot description, URDF)
Before this commit: robot left_gripper_v2_final, 14 links, 13 joints
Links:
- removed link controller_holder
Joints:
- removed joint controller_holder_frame

File: assets/yubi_description/source/yubi_right_gripper.urdf (robot description, URDF)
Before this commit: robot right_gripper_corrected_fixed, 14 links, 13 joints
Links:
- removed link controller_holder
Joints:
- removed joint controller_holder_frame

File: assets/yubi_description/urdf/yubi_hands.urdf (robot description, URDF)
Before this commit: robot yubi_hands, 31 links, 30 joints
Links:
- removed link left_controller_holder
- removed link right_controller_holder
Joints:
- removed joint left_controller_holder_frame
- removed joint right_controller_holder_frame
