Commit message: E5: the calibration library, and the humanoid's head camera declared
sx_embodiments.calibrate (the calibrate extra: NumPy, SciPy, OpenCV) measures a built
robot into the calibration kinds. solve_intrinsics fits a camera unit's lens from
checkerboard or ChArUco views; solve_mounts places cameras on the links that carry them
from views of a target another link holds, one model for eye-in-hand, eye-to-base, a
head camera watching a hand-held target and a tracked rig over a static board, cameras
that saw one target solved together and a checkerboard's half-turn order resolved per
view. measure_intrinsics and measure_mount bind both to a robot instance: the unit in
the camera's slot, the body's raster, every view's transform from forward kinematics
over the body's own description at the recorded joint positions.

sx_embodiments.kinematics is the one URDF chain reader (fixed, revolute, continuous,
prismatic, mimic; floating and planar parsed and refused on a path), and the humanoid
tests use it.

The humanoid upper body and full humanoid declare the head's RealSense D435 colour
stream at 1280x720 with the datasheet's nominal optics (Intel 337029-009, OV2740 field
of view) on a new head_camera_color_optical frame at the CAD camera origin. Assembly
frames can declare the camera_optical convention. Both humanoid ids move (pinned);
previews re-keyed; the Damiao transcripts re-minted from DM_CAN.py with every wire byte
unchanged (only the bindings id moved).

Co-Authored-By: Claude Opus 5.5 <noreply@anthropic.com>

File: assets/humanoid_pkg/urdf/sentient_humanoid.urdf (robot description, URDF)
Before this commit: robot sentient_humanoid, 42 links, 41 joints
Links:
- added link head_camera_color_optical
Joints:
- added joint camera_link_to_head_camera_color_optical: type fixed, parent camera_link, child head_camera_color_optical, origin xyz=0 0 0 rpy=-1.5707963267948966 0 -1.5707963267948966

File: assets/humanoid_pkg/urdf/sentient_humanoid_upper_body.urdf (robot description, URDF)
Before this commit: robot sentient_humanoid_upper_body, 24 links, 23 joints
Links:
- added link head_camera_color_optical
Joints:
- added joint camera_link_to_head_camera_color_optical: type fixed, parent camera_link, child head_camera_color_optical, origin xyz=0 0 0 rpy=-1.5707963267948966 0 -1.5707963267948966
