Commit message: The Omron LD under panda_omron is robosuite's own meshes, and its earlier identity still resolves
The Omron LD module is now robosuite's omron_mobile_base: its eight meshes and the MJCF
copied byte for byte at a pinned commit with the MIT licence in the directory, and a
first-party URDF projection of the wheeled base and support column that the module
describes itself with. panda_omron renders the Panda on it as robosuite builds PandaOmron.

A body's definition now names the identities of its earlier revisions under the current
schema; the registry answers one with the revision that superseded it, so RoboCasa
recordings that name panda_omron before its base was drawn still find their body.

Co-Authored-By: Claude Opus 5.5 <noreply@anthropic.com>

File: assets/official/franka_panda/panda_omron.urdf (robot description, URDF)
Before this commit: robot panda_omron, 24 links, 23 joints
Links:
- link omron_ld: geometry collision box size=0.7 0.5 0.38; collision cylinder length=0.4 radius=0.12
