Commit message: Take the static upper body's motor table and confirmed limits
Subraj's revised description adds the robot's Damiao motor table: per torso and
arm joint the model, CAN send and answer ids, MIT gains, limits, and flags that
mapping, direction and limits are confirmed on the robot. Kinematics and meshes
are unchanged.

The torso and both arms are now direct Damiao drives with actuator feedback,
bound from that table (forearm yaw is a DM4340), and a test holds the bindings
equal to it. The rendering no longer moves the elbow range or cuts forearm yaw
to one turn: the elbow is an offset joint bending both ways about the hanging
forearm, and both ranges are the robot's confirmed stops. The motor table is
dropped from the simulation description, since the bindings carry it. It stays
a development body while its masses are hull estimates.

Co-Authored-By: Claude Opus 5.5 <noreply@anthropic.com>

File: assets/sentient_static_upper_body/sentient_static_upper_body.urdf (robot description, URDF)
Before this commit: robot sentient_static_upper_body, 33 links, 32 joints
Joints:
- joint left_elbow_pitch_joint: limit lower=-1.57079632679 upper=1.17920367321 effort=54 velocity=0.5 -> lower=-2.9753185320820936 upper=0.000953688868543523 effort=54 velocity=0.5
- joint left_forearm_yaw_joint: limit lower=-3.14159265359 upper=1.88391699092 effort=54 velocity=0.5 -> lower=-6.82669565880827 upper=1.8839169909208824 effort=54 velocity=0.5
- joint left_gripper_left_finger_joint: limit lower=-0.823747683095 upper=0 effort=1 velocity=1 -> lower=-0.8237476830945893 upper=0.0 effort=1 velocity=1
- joint left_gripper_right_finger_joint: limit lower=0 upper=0.929592357459 effort=1 velocity=1 -> lower=0.0 upper=0.9295923574586985 effort=1 velocity=1
- joint left_shoulder_pitch_joint: limit lower=-2.64267185473 upper=2.88986800946 effort=54 velocity=0.5 -> lower=-2.642671854734111 upper=2.889868009460594 effort=54 velocity=0.5
- joint left_shoulder_roll_joint: limit lower=-0.387388418402 upper=1.20183871214 effort=54 velocity=0.5 -> lower=-0.3873884184023808 upper=1.2018387121385512 effort=54 velocity=0.5
- joint left_upper_arm_yaw_joint: limit lower=-5.12302586404 upper=0.807011520562 effort=54 velocity=0.5 -> lower=-5.1230258640421145 upper=0.8070115205615327 effort=54 velocity=0.5
- joint left_wrist_pitch_joint: limit lower=-2.12806134127 upper=2.44087129015 effort=54 velocity=0.5 -> lower=-2.1280613412680243 upper=2.4408712901503016 effort=54 velocity=0.5
- joint left_wrist_roll_joint: limit lower=-2.09601739528 upper=2.09678034638 effort=54 velocity=0.5 -> lower=-2.096017395284962 upper=2.0967803463797967 effort=54 velocity=0.5
- joint right_elbow_pitch_joint: limit lower=-1.17920367321 upper=1.57079632679 effort=54 velocity=0.5 -> lower=-0.029182879377431803 upper=2.966544594491493 effort=54 velocity=0.5
- joint right_forearm_yaw_joint: limit lower=-3.14159265359 upper=1.42614633402 effort=54 velocity=0.5 -> lower=-6.009575036240177 upper=1.4261463340199896 effort=54 velocity=0.5
- joint right_gripper_left_finger_joint: limit lower=-0.952602069277 upper=0 effort=1 velocity=1 -> lower=-0.9526020692769832 upper=0.0 effort=1 velocity=1
- joint right_gripper_right_finger_joint: limit lower=0 upper=0.788466124973 effort=1 velocity=1 -> lower=0.0 upper=0.7884661249732196 effort=1 velocity=1
- joint right_shoulder_pitch_joint: limit lower=-2.91390096895 upper=3.12256809339 effort=54 velocity=0.5 -> lower=-2.9139009689478907 upper=3.1225680933852136 effort=54 velocity=0.5
- joint right_shoulder_roll_joint: limit lower=-1.21010342679 upper=0.354649110181 effort=54 velocity=0.5 -> lower=-1.2101034267894413 upper=0.35464911018127765 effort=54 velocity=0.5
- joint right_upper_arm_yaw_joint: limit lower=-2.42103456168 upper=2.75978484779 effort=54 velocity=0.5 -> lower=-2.4210345616845963 upper=2.7597848477912574 effort=54 velocity=0.5
- joint right_wrist_pitch_joint: limit lower=-2.30888075074 upper=2.25585564965 effort=54 velocity=0.5 -> lower=-2.308880750743878 upper=2.255855649652858 effort=54 velocity=0.5
- joint right_wrist_roll_joint: limit lower=-2.11203936828 upper=2.09868772412 effort=54 velocity=0.5 -> lower=-2.112039368276493 upper=2.0986877241168838 effort=54 velocity=0.5
- joint so101_camera_tilt_joint: limit lower=-0.106465084372 upper=2.04203522483 effort=1 velocity=1 -> lower=-0.10646508437165425 upper=2.0420352248333655 effort=1 velocity=1
- joint so101_elbow_flex_joint: limit lower=-3.40339204139 upper=0.0872664625997 effort=1 velocity=1 -> lower=-3.403392041388943 upper=0.08726646259971617 effort=1 velocity=1
- joint so101_shoulder_lift_joint: limit lower=-0.0349065850399 upper=3.63028484415 effort=1 velocity=1 -> lower=-0.03490658503988664 upper=3.6302848441482056 effort=1 velocity=1
- joint so101_shoulder_pan_joint: limit lower=-2.12930168743 upper=2.12930168743 effort=1 velocity=1 -> lower=-2.129301687433082 upper=2.1293016874330815 effort=1 velocity=1
- joint so101_wrist_flex_joint: limit lower=-3.28121899375 upper=0.401425727959 effort=1 velocity=1 -> lower=-3.2812189937493397 upper=0.4014257279586958 effort=1 velocity=1
- joint so101_wrist_roll_joint: limit lower=-3.00196631343 upper=2.86233997327 effort=1 velocity=1 -> lower=-3.001966313430247 upper=2.8623399732707 effort=1 velocity=1
- joint torso_joint: limit lower=-1.22129396506 upper=1.14995803769 effort=54 velocity=0.5 -> lower=-1.221293965056839 upper=1.1499580376897836 effort=54 velocity=0.5

File: assets/sentient_static_upper_body/source/received.urdf (robot description, URDF)
Before this commit: robot allisa_calibrated_feedback, 34 links, 33 joints
Links:
- link base_link: geometry visual mesh filename=package://humanoid_pkg/models/allisa_current/meshes_preview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 scale=1 1 1; visual mesh filename=package://humanoid_pkg/models/allisa_current/meshes_preview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 scale=1 1 1
- link camera_link: geometry visual mesh filename=package://humanoid_pkg/models/allisa_current/meshes_preview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 scale=1 1 1; visual mesh filename=package://humanoid_pkg/models/allisa_current/meshes_preview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 scale=1 1 1
- link chest_link: geometry visual mesh filename=package://humanoid_pkg/models/allisa_current/meshes_preview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 scale=1 1 1; visual mesh filename=package://humanoid_pkg/models/allisa_current/meshes_preview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 scale=1 1 1
- link left_elbow_pitch_link: geometry visual mesh filename=package://humanoid_pkg/models/allisa_current/meshes_preview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 scale=1 1 1; visual mesh filename=package://humanoid_pkg/models/allisa_current/meshes_preview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 scale=1 1 1
- link left_forearm_yaw_link: geometry collision cylinder length=0.19939090307297475 radius=0.027; collision sphere radius=0.027
- link left_gripper_base_link: geometry visual mesh filename=package://humanoid_pkg/models/allisa_current/meshes_preview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 scale=1 1 1; visual mesh filename=package://humanoid_pkg/models/allisa_current/meshes_preview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 scale=1 1 1
- link left_gripper_left_finger_link: geometry visual mesh filename=package://humanoid_pkg/models/allisa_current/meshes_preview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 scale=1 1 1; visual mesh filename=package://humanoid_pkg/models/allisa_current/meshes_preview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 scale=1 1 1
- link left_gripper_right_finger_link: geometry visual mesh filename=package://humanoid_pkg/models/allisa_current/meshes_preview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 scale=1 1 1; visual mesh filename=package://humanoid_pkg/models/allisa_current/meshes_preview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 scale=1 1 1
- link left_shoulder_pitch_link: geometry visual mesh filename=package://humanoid_pkg/models/allisa_current/meshes_preview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 scale=1 1 1; visual mesh filename=package://humanoid_pkg/models/allisa_current/meshes_preview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 scale=1 1 1
- link left_shoulder_roll_link: geometry visual mesh filename=package://humanoid_pkg/models/allisa_current/meshes_preview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 scale=1 1 1; visual mesh filename=package://humanoid_pkg/models/allisa_current/meshes_preview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 scale=1 1 1
- link left_upper_arm_yaw_link: geometry collision cylinder length=0.212639633100138 radius=0.027; collision sphere radius=0.027
- link left_wrist_pitch_link: geometry collision cylinder length=0.09767557839074484 radius=0.027; collision sphere radius=0.027
- link left_wrist_roll_link: geometry collision cylinder length=0.15152229474162202 radius=0.025; collision sphere radius=0.025
- link right_elbow_pitch_link: geometry visual mesh filename=package://humanoid_pkg/models/allisa_current/meshes_preview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 scale=1 1 1; visual mesh filename=package://humanoid_pkg/models/allisa_current/meshes_preview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 scale=1 1 1
- link right_forearm_yaw_link: geometry collision cylinder length=0.1897229826655043 radius=0.027; collision sphere radius=0.027
- link right_gripper_base_link: geometry visual mesh filename=package://humanoid_pkg/models/allisa_current/meshes_preview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 scale=1 1 1; visual mesh filename=package://humanoid_pkg/models/allisa_current/meshes_preview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 scale=1 1 1
- link right_gripper_left_finger_link: geometry visual mesh filename=package://humanoid_pkg/models/allisa_current/meshes_preview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 scale=1 1 1; visual mesh filename=package://humanoid_pkg/models/allisa_current/meshes_preview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 scale=1 1 1
- link right_gripper_right_finger_link: geometry visual mesh filename=package://humanoid_pkg/models/allisa_current/meshes_preview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 scale=1 1 1; visual mesh filename=package://humanoid_pkg/models/allisa_current/meshes_preview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 scale=1 1 1
- link right_shoulder_pitch_link: geometry visual mesh filename=package://humanoid_pkg/models/allisa_current/meshes_preview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 scale=1 1 1; visual mesh filename=package://humanoid_pkg/models/allisa_current/meshes_preview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 scale=1 1 1
- link right_shoulder_roll_link: geometry visual mesh filename=package://humanoid_pkg/models/allisa_current/meshes_preview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 scale=1 1 1; visual mesh filename=package://humanoid_pkg/models/allisa_current/meshes_preview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 scale=1 1 1
- link right_upper_arm_yaw_link: geometry collision cylinder length=0.21592472264460436 radius=0.027; collision sphere radius=0.027
- link right_wrist_pitch_link: geometry collision cylinder length=0.09767557839072052 radius=0.027; collision sphere radius=0.027
- link right_wrist_roll_link: geometry collision cylinder length=0.1515238794754327 radius=0.025; collision sphere radius=0.025
- link so101_base_link: geometry visual mesh filename=package://humanoid_pkg/models/allisa_current/meshes_preview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 scale=1 1 1; visual mesh filename=package://humanoid_pkg/models/allisa_current/meshes_preview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 scale=1 1 1
- link so101_elbow_flex_link: geometry visual mesh filename=package://humanoid_pkg/models/allisa_current/meshes_preview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 scale=1 1 1; visual mesh filename=package://humanoid_pkg/models/allisa_current/meshes_preview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 scale=1 1 1
- link so101_shoulder_lift_link: geometry visual mesh filename=package://humanoid_pkg/models/allisa_current/meshes_preview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 scale=1 1 1; visual mesh filename=package://humanoid_pkg/models/allisa_current/meshes_preview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 scale=1 1 1
- link so101_shoulder_pan_link: geometry visual mesh filename=package://humanoid_pkg/models/allisa_current/meshes_preview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 scale=1 1 1; visual mesh filename=package://humanoid_pkg/models/allisa_current/meshes_preview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 scale=1 1 1
- link so101_wrist_flex_link: geometry visual mesh filename=package://humanoid_pkg/models/allisa_current/meshes_preview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 scale=1 1 1; visual mesh filename=package://humanoid_pkg/models/allisa_current/meshes_preview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 scale=1 1 1
- link so101_wrist_roll_link: geometry visual mesh filename=package://humanoid_pkg/models/allisa_current/meshes_preview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 scale=1 1 1; visual mesh filename=package://humanoid_pkg/models/allisa_current/meshes_preview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 scale=1 1 1
- link torso_link: geometry collision box size=.13 .19 .33; visual mesh filename=package://humanoid_pkg/models/allisa_current/meshes_preview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 scale=1 1 1

Commit message: Register the static upper body's ZED 2i head camera and capture it as one stereo track
The ZED 2i on the SO-101 neck becomes two declared cameras, head_left and
head_right, on optical frames the description rendering adds 60 mm either side
of ZED_camera (the frame's meshes put the lens barrels there, looking along +x).
They publish as one side-by-side head track at HD720 and 30 fps.

zed_2i joins the camera vocabulary. factory_intrinsics.zed_factory_calibration
reads the per-serial factory ini Stereolabs publishes (calib.stereolabs.com):
each eye's rational 8-term lens, and the right eye's pose in the left's frame.
Unit 30371653's record is the fixture. The registry re-renders the URDF, asset
manifest, bindings, drives, media plans and poses, plus a new sx-uvc-stereo
plan with the unit placed and calibrated.

drivers/sx-uvc-stereo turns that track into a CaptureRequest and splits each
YUYV side-by-side frame into two I420 eyes. Behind the capture feature it opens
the device through nokhwa (V4L2, AVFoundation), by sysfs serial on Linux.

Co-Authored-By: Claude Opus 5.5 <noreply@anthropic.com>

File: assets/sentient_static_upper_body/sentient_static_upper_body.urdf (robot description, URDF)
Before this commit: robot sentient_static_upper_body, 33 links, 32 joints
Links:
- added link zed_left_optical
- added link zed_right_optical
Joints:
- added joint ZED_camera_to_zed_left_optical: type fixed, parent ZED_camera, child zed_left_optical, origin xyz=0 0.06 0 rpy=-1.5707963267948966 0 -1.5707963267948966
- added joint ZED_camera_to_zed_right_optical: type fixed, parent ZED_camera, child zed_right_optical, origin xyz=0 -0.06 0 rpy=-1.5707963267948966 0 -1.5707963267948966

Commit message: Describe the static upper body from allisa_bot, the operator-selected model
humanoid_pkg's notes of 2026-10-25 say the operator rejected the
allisa_feedback geometry this body was registered from and selected
urdf/allisa_bot.urdf; the feedback model is a joint-limit donor only. That
file is now the source, byte for byte (sha256 039b0b7d), with the package's
169 display meshes and its integration notes, model provenance, hardware
profile and Feetech record. received.urdf and its decimated meshes leave the
tree and stay in history.

allisa_bot matches the feedback file on every link, visual and joint origin,
neck included. It reverses both wrist axes on each arm, has no collisions,
and carries zed2i_left_optical_frame instead of ZED_camera. The rendering
adds hull collisions and inertials, unique visual names, meshes/ paths and
drops the Gazebo sensor element. It negates the four wrist limits, which the
donor gives in motor coordinates. It places ZED_camera so the registry's left
eye is the source's optical frame; that swaps left and right relative to the
old ZED_camera.

The arm bindings are the hardware profile: the same ids, models and gains as
the old motor table, with both wrists at sign -1. The torso, absent from the
profile, keeps the old table's 0x1F. The gripper sides and ids match the
Feetech record's board serials. Tests hold the bindings to the profile and
every source joint to the rendering, and the left eye to the source frame.

Co-Authored-By: Claude Opus 5.5 <noreply@anthropic.com>

File: assets/sentient_static_upper_body/sentient_static_upper_body.urdf (robot description, URDF)
Before this commit: robot sentient_static_upper_body, 35 links, 34 joints
Links:
- added link zed2i_left_optical_frame
- link base_link: mass 1.50434 -> 1.45907; geometry collision mesh filename=meshes/collision/base_link.stl; visual mesh filename=meshes/_________step__Body1_1_.stl scale=1 1 1
- link camera_link: mass 0.263961 -> 0.264253; geometry collision mesh filename=meshes/collision/camera_link.stl; visual mesh filename=meshes/Camera_Component___Body___ZED_2i___4_6mm___Cover_ste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 scale=1 1 1
- link chest_link: mass 4.80853 -> 4.79762; geometry collision mesh filename=meshes/collision/chest_link.stl; visual mesh filename=meshes/J8009P_2EC_RAU_5005______20240809_stp__NONE.stl scale=1 1 1
- link left_elbow_pitch_link: mass 0.134107 -> 0.133283; geometry collision mesh filename=meshes/collision/left_elbow_pitch_link.stl; visual mesh filename=meshes/bearing_fl6803zz.stl scale=1 1 1
- link left_forearm_yaw_link: mass 0.261966 -> 0.263184; geometry collision mesh filename=meshes/collision/left_forearm_yaw_link.stl; visual mesh filename=meshes/DM_J4310_2EC_V1_1__3d_20240822_1__DM_J4310_2EC_V1_1_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 scale=1 1 1
- link left_gripper_base_link: mass 0.0481413 -> 0.048405; geometry collision mesh filename=meshes/collision/left_gripper_base_link.stl; visual mesh filename=meshes/GE_27_2_step____1_1_.stl scale=1 1 1
- link left_gripper_left_finger_link: mass 0.0266942 -> 0.0271797; geometry collision mesh filename=meshes/collision/left_gripper_left_finger_link.stl; visual mesh filename=meshes/_________2_step____1_1_.stl scale=1 1 1
- link left_gripper_right_finger_link: mass 0.026693 -> 0.0271687; geometry collision mesh filename=meshes/collision/left_gripper_right_finger_link.stl; visual mesh filename=meshes/_________2_step____1_1_.stl scale=1 1 1
- link left_shoulder_pitch_link: mass 0.346796 -> 0.346967; geometry collision mesh filename=meshes/collision/left_shoulder_pitch_link.stl; visual mesh filename=meshes/J8009P_2EC_RAU_5005______20240809_stp__NONE.stl scale=1 1 1
- link left_shoulder_roll_link: mass 0.364166 -> 0.360351; geometry collision mesh filename=meshes/collision/left_shoulder_roll_link.stl; visual mesh filename=meshes/dm_4340P_20250407_1_stp__dm_4340P_20250407_1_stp_1__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 scale=1 1 1
- link left_upper_arm_yaw_link: mass 0.181482 -> 0.181364; geometry collision mesh filename=meshes/collision/left_upper_arm_yaw_link.stl; visual mesh filename=meshes/bicep_yaw_to_elbow_bracket_1.stl scale=1 1 1
- link left_wrist_pitch_link: mass 0.14067 -> 0.141803; geometry collision mesh filename=meshes/collision/left_wrist_pitch_link.stl; visual mesh filename=meshes/DM_J4310_2EC_V1_1__3d_20240822_1__DM_J4310_2EC_V1_1_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 scale=1 1 1
- link left_wrist_roll_link: mass 0.202201 -> 0.2007; geometry collision mesh filename=meshes/collision/left_wrist_roll_link.stl; visual mesh filename=meshes/BRACKET_CAMERA.stl scale=1 1 1
- link right_elbow_pitch_link: mass 0.134107 -> 0.133283; geometry collision mesh filename=meshes/collision/right_elbow_pitch_link.stl; visual mesh filename=meshes/bearing_fl6803zz.stl scale=1 1 1
- link right_forearm_yaw_link: mass 0.261968 -> 0.262855; geometry collision mesh filename=meshes/collision/right_forearm_yaw_link.stl; visual mesh filename=meshes/DM_J4310_2EC_V1_1__3d_20240822_1__DM_J4310_2EC_V1_1_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 scale=1 1 1
- link right_gripper_base_link: mass 0.0481414 -> 0.0484051; geometry collision mesh filename=meshes/collision/right_gripper_base_link.stl; visual mesh filename=meshes/GE_27_2_step____1_1_.stl scale=1 1 1
- link right_gripper_left_finger_link: mass 0.0266942 -> 0.0271797; geometry collision mesh filename=meshes/collision/right_gripper_left_finger_link.stl; visual mesh filename=meshes/_________2_step____1_1_.stl scale=1 1 1
- link right_gripper_right_finger_link: mass 0.026693 -> 0.0271687; geometry collision mesh filename=meshes/collision/right_gripper_right_finger_link.stl; visual mesh filename=meshes/_________2_step____1_1_.stl scale=1 1 1
- link right_shoulder_pitch_link: mass 0.346796 -> 0.346981; geometry collision mesh filename=meshes/collision/right_shoulder_pitch_link.stl; visual mesh filename=meshes/J8009P_2EC_RAU_5005______20240809_stp__NONE.stl scale=1 1 1
- link right_shoulder_roll_link: mass 0.366383 -> 0.362339; geometry collision mesh filename=meshes/collision/right_shoulder_roll_link.stl; visual mesh filename=meshes/dm_4340P_20250407_1_stp__dm_4340P_20250407_1_stp_1__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 scale=1 1 1
- link right_upper_arm_yaw_link: mass 0.181482 -> 0.181364; geometry collision mesh filename=meshes/collision/right_upper_arm_yaw_link.stl; visual mesh filename=meshes/bicep_yaw_to_elbow_bracket_1.stl scale=1 1 1
- link right_wrist_pitch_link: mass 0.14067 -> 0.141803; geometry collision mesh filename=meshes/collision/right_wrist_pitch_link.stl; visual mesh filename=meshes/DM_J4310_2EC_V1_1__3d_20240822_1__DM_J4310_2EC_V1_1_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 scale=1 1 1
- link right_wrist_roll_link: mass 0.202201 -> 0.2007; geometry collision mesh filename=meshes/collision/right_wrist_roll_link.stl; visual mesh filename=meshes/BRACKET_CAMERA.stl scale=1 1 1
- link so101_base_link: mass 0.28733 -> 0.288892; geometry collision mesh filename=meshes/collision/so101_base_link.stl; visual mesh filename=meshes/Base_08p_step__Body4_1_.stl scale=1 1 1
- link so101_elbow_flex_link: mass 0.179963 -> 0.180313; geometry collision mesh filename=meshes/collision/so101_elbow_flex_link.stl; visual mesh filename=meshes/GE_27_step__Body1_1_.stl scale=1 1 1
- link so101_shoulder_lift_link: mass 0.193778 -> 0.194153; geometry collision mesh filename=meshes/collision/so101_shoulder_lift_link.stl; visual mesh filename=meshes/GE_27_step__Body1_1_.stl scale=1 1 1
- link so101_shoulder_pan_link: mass 0.134083 -> 0.134995; geometry collision mesh filename=meshes/collision/so101_shoulder_pan_link.stl; visual mesh filename=meshes/GE_27_step__Body1_1_.stl scale=1 1 1
- link so101_wrist_flex_link: mass 0.0706334 -> 0.0703263; geometry collision mesh filename=meshes/collision/so101_wrist_flex_link.stl; visual mesh filename=meshes/GE_27_step__Body1_1_.stl scale=1 1 1
- link so101_wrist_roll_link: mass 0.0508075 -> 0.0509793; geometry collision mesh filename=meshes/collision/so101_wrist_roll_link.stl; visual mesh filename=meshes/GE_27_step__Body1_1_.stl scale=1 1 1
- link torso_link: mass 0.629743 -> 0.634213; geometry collision mesh filename=meshes/collision/torso_link.stl; visual mesh filename=meshes/J8009P_2EC_RAU_5005______20240809_stp__NONE.stl scale=1 1 1
Joints:
- removed joint camera_link_to_ZED_camera
- added joint zed2i_left_optical_frame_to_ZED_camera: type fixed, parent zed2i_left_optical_frame, child ZED_camera, origin xyz=0.06 0 0 rpy=0.785398163 -1.57079633 0.785398163
- added joint zed2i_left_optical_joint: type fixed, parent camera_link, child zed2i_left_optical_frame, origin xyz=-0.0426184 -0.0431015 0.0795497 rpy=3.14159265359 1.57079632679 0
- joint left_wrist_pitch_joint: axis 3.54287553479e-05 0.99999999937 -1.97553215478e-06 -> -3.54287553479e-05 -0.99999999937 1.97553215478e-06; limit lower=-2.1280613412680243 upper=2.4408712901503016 effort=54 velocity=0.5 -> lower=-2.4408712901503016 upper=2.1280613412680243 effort=54 velocity=0.5
- joint left_wrist_roll_joint: axis 0.99999999925 -3.54287862224e-05 -1.56307773885e-05 -> -0.99999999925 3.54287862224e-05 1.56307773885e-05; limit lower=-2.096017395284962 upper=2.0967803463797967 effort=54 velocity=0.5 -> lower=-2.0967803463797967 upper=2.096017395284962 effort=54 velocity=0.5
- joint right_wrist_pitch_joint: axis -1.62246979482e-05 -0.999999999813 1.04829448668e-05 -> 1.62246979482e-05 0.999999999813 -1.04829448668e-05; limit lower=-2.308880750743878 upper=2.255855649652858 effort=54 velocity=0.5 -> lower=-2.255855649652858 upper=2.308880750743878 effort=54 velocity=0.5
- joint right_wrist_roll_joint: axis 0.999999999854 -1.62246422642e-05 5.31185315207e-06 -> -0.999999999854 1.62246422642e-05 -5.31185315207e-06; limit lower=-2.112039368276493 upper=2.0986877241168838 effort=54 velocity=0.5 -> lower=-2.0986877241168838 upper=2.112039368276493 effort=54 velocity=0.5
