Commit message: Put the official new-calibration SO-101 under the static upper body's neck
The owner reports allisa_bot's SO-101 breaks apart and self-collides, and it
is the feedback file's CAD export: arbitrary joint zeros, links 15 to 29 mm
off along the pitch axes, and at its own zero pose it penetrates the robot.
From so101_shoulder_pan_joint down the neck is now TheRobotStudio's
so101_new_calib chain (SO-ARM100 5f6d2b8, Apache-2.0), vendored byte for byte
with its meshes. Its zeros are LeRobot's calibrated mid-range, so neck
readings need no offsets.

allisa_bot's own base, its holder for the camera servo, the camera bracket and
the ZED 2i meshes ride on the official chain, each placed by registering the
official parts onto allisa_bot's CAD (0.4 to 0.9 mm rms). The base turns half
a turn, as the robot is built. With zero offsets the recording at the side
photo reproduces the side, front and rear photos. The bracket's angle on the
tilt servo's horn is fitted to the side photo. The camera tilt keeps the
official joint's origin and axis but declares the free arc it rests in
(-180 to -15 deg), because the bracket meets the wrist between about +10 and
+130 deg. Its home is its recorded rest.

A MuJoCo contact check of the rendered collisions is clean at the zero and
recorded rest poses. Tests hold the neck to the official file and every other
link and joint to allisa_bot. The neck bring-in tests take the new ranges.

Co-Authored-By: Claude Opus 5.5 <noreply@anthropic.com>

File: assets/sentient_static_upper_body/sentient_static_upper_body.urdf (robot description, URDF)
Before this commit: robot sentient_static_upper_body, 36 links, 35 joints
Links:
- link so101_elbow_flex_link: mass 0.180313 -> 0.104; geometry collision mesh filename=meshes/so101/motor_holder_so101_wrist_v1.stl; collision mesh filename=meshes/so101/sts3215_03a_v1.stl
- link so101_shoulder_lift_link: mass 0.194153 -> 0.103; geometry collision mesh filename=meshes/so101/sts3215_03a_v1.stl; collision mesh filename=meshes/so101/upper_arm_so101_v1.stl
- link so101_shoulder_pan_link: mass 0.134995 -> 0.100006; geometry collision mesh filename=meshes/so101/motor_holder_so101_base_v1.stl; collision mesh filename=meshes/so101/rotation_pitch_so101_v1.stl
- link so101_wrist_flex_link: mass 0.0703263 -> 0.079; geometry collision mesh filename=meshes/so101/sts3215_03a_no_horn_v1.stl; collision mesh filename=meshes/so101/wrist_roll_pitch_so101_v2.stl
- link so101_wrist_roll_link: mass 0.0509793 -> 0.087; geometry collision mesh filename=meshes/Wrist_Roll_Follower_SO101_5__Fillet1.stl; collision mesh filename=meshes/so101/sts3215_03a_v1.stl
Joints:
- joint so101_camera_tilt_joint: limit lower=-0.10646508437165425 upper=2.0420352248333655 effort=1 velocity=1 -> lower=-3.14159265 upper=-0.261799388 effort=10 velocity=10; origin xyz=0.0202 0.0221559269193 -0.023399987673 rpy=1.57080005267 0.168347452146 6.24283662386e-07 -> xyz=0.0202 0.0188 -0.0234 rpy=1.5708 -5.24284e-08 -1.41553e-15
- joint so101_elbow_flex_joint: limit lower=-3.403392041388943 upper=0.08726646259971617 effort=1 velocity=1 -> lower=-1.69 upper=1.69 effort=10 velocity=10; origin xyz=-0.11257 -0.028 0.0191075992233 rpy=8.69253632799e-16 4.4408920985e-16 3.12605992077 -> xyz=-0.11257 -0.028 1.73763e-16 rpy=-3.63608e-16 8.74301e-16 1.5708
- joint so101_mount_joint: origin xyz=-0.0916244982412 0.123363123582 0.0523846737825 rpy=0 0 0 -> xyz=-0.0347334982 0.0916071236 0.0471956738 rpy=0 -0 3.14159265
- joint so101_shoulder_lift_joint: limit lower=-0.03490658503988664 upper=3.6302848441482056 effort=1 velocity=1 -> lower=-1.74533 upper=1.74533 effort=10 velocity=10; origin xyz=-0.0303991433191 -0.00284688859968 -0.0541999999998 rpy=1.57079632678 0.337616266773 3.14158898038 -> xyz=-0.0303992 -0.0182778 -0.0542 rpy=-1.5708 -1.5708 0
- joint so101_shoulder_pan_joint: limit lower=-2.129301687433082 upper=2.1293016874330815 effort=1 velocity=1 -> lower=-1.91986 upper=1.91986 effort=10 velocity=10; origin xyz=0.053194105349 -0.0318758054314 0.0577853490004 rpy=-3.14142530718 -0.00872519 3.12334 -> xyz=0.0388353 -8.97657e-09 0.0624 rpy=3.14159 4.18253e-17 -3.14159
- joint so101_wrist_flex_joint: limit lower=-3.2812189937493397 upper=0.4014257279586958 effort=1 velocity=1 -> lower=-1.65806 upper=1.65806 effort=10 velocity=10; origin xyz=-0.1349 0.0052 -0.0288327991411 rpy=1.83316892365e-15 -3.5527136788e-15 -0.249320445083 -> xyz=-0.1349 0.0052 3.62355e-17 rpy=4.02456e-15 8.67362e-16 -1.5708
- joint so101_wrist_roll_joint: limit lower=-3.001966313430247 upper=2.8623399732707 effort=1 velocity=1 -> lower=-2.74385 upper=2.84121 effort=10 velocity=10; origin xyz=-1.14828424547e-09 -0.0615054204925 0.0181000014874 rpy=1.57079999957 0.0461946780963 3.14158999086 -> xyz=5.55112e-17 -0.0611 0.0181 rpy=1.5708 0.0486795 3.14159
- joint zed2i_left_optical_joint: origin xyz=-0.0426184 -0.0431015 0.0795497 rpy=3.14159265359 1.57079632679 0 -> xyz=0.0492377082 0.0353513141 0.0761937731 rpy=-2.63392831 1.57079633 -2.80227582

Commit message: Static upper body: SO-101 base faces as allisa_bot places it; camera mount angle from the ZED IMU
The operator at the robot saw the SO-101 base facing backwards in the twin, so the half turn
about the base plate centre is removed. CAMERA_MOUNT_TILT is half a turn plus 141.56 deg,
solved so the model's camera tilt matches the ZED 2i IMU's gravity reading (2.3 deg residual at
one neck pose, 0.35 deg pitch at a second; a +114 tick tilt step moved the IMU 9.8 deg).

Known wrong, open: with these the model's camera faces backwards (heading 177 deg) and tipped
up, while the operator sees it facing forward and tipped slightly down. Gravity cannot see
heading, and the operator's view suggests the IMU's pitch sign in sx-stereolabs-sensors is
reversed, which would make the tilt fit wrong too. Suspects: the IMU axis mapping, and the
wrist roll servo's zero (a half turn of so101_wrist_roll_joint turns the camera forward).

Co-Authored-By: Claude Opus 5.5 <noreply@anthropic.com>

File: assets/sentient_static_upper_body/sentient_static_upper_body.urdf (robot description, URDF)
Before this commit: robot sentient_static_upper_body, 36 links, 35 joints
Joints:
- joint so101_mount_joint: origin xyz=-0.0347334982 0.0916071236 0.0471956738 rpy=0 -0 3.14159265 -> xyz=-0.0777334982 0.0916071236 0.0471956738 rpy=0 -0 0
- joint zed2i_left_optical_joint: origin xyz=0.0492377082 0.0353513141 0.0761937731 rpy=-2.63392831 1.57079633 -2.80227582 -> xyz=-0.0605436352 0.00292156772 0.0761937731 rpy=2.82847395 1.57079633 -1.15237077

Commit message: Static upper body: the camera faces forward, slightly down, as on the robot
#61 left the model's camera facing backwards into the wrist (heading 177 deg) and tipped up;
the operator sees it facing forward and slightly down. The received holder sits half a turn
round the wrist roll horn from the official fixed jaw (CAMERA_ROLL_TURN), which turns the
camera forward (heading -2.9 deg), and CAMERA_MOUNT_TILT is re-solved to put it 7.95 deg nose
down at the recorded pose, the IMU's tilt magnitude. The IMU tool reported that pose as nose
up, so its pitch sign is suspect and the tilt joint's sense is unconfirmed; both are open.

Co-Authored-By: Claude Opus 5.5 <noreply@anthropic.com>

File: assets/sentient_static_upper_body/sentient_static_upper_body.urdf (robot description, URDF)
Before this commit: robot sentient_static_upper_body, 36 links, 35 joints
Joints:
- joint so101_camera_tilt_joint: origin xyz=0.0202 0.0188 -0.0234 rpy=1.5708 -5.24284e-08 -1.41553e-15 -> xyz=-0.0202 -0.0188 -0.0234 rpy=1.5708 -5.24284e-08 3.14159265
- joint zed2i_left_optical_joint: origin xyz=-0.0605436352 0.00292156772 0.0761937731 rpy=2.82847395 1.57079633 -1.15237077 -> xyz=-0.05875235 -0.0149073367 0.0761937731 rpy=2.73522519 1.57079633 -0.948913556

Commit message: Static upper body: the camera turns only about its tilt axis; undo the wrist roll half turn
#63 turned the camera holder half a turn round the wrist roll horn, which the holder cannot
do, and left a part floating beside the camera. The holder stays as built; the camera turns
only about the tilt axis, and CAMERA_MOUNT_TILT puts the ZED body upright, facing forward and
7.8 deg nose down at the recorded pose, as on the robot and in the side photo.

Open: at this angle the ZED_camera frame is upside down against the ZED meshes, so that frame
(built from allisa_bot's left optical frame) and the IMU mounted on it carry a convention
error, which is why the IMU's reported pitch sign was wrong.

Co-Authored-By: Claude Opus 5.5 <noreply@anthropic.com>

File: assets/sentient_static_upper_body/sentient_static_upper_body.urdf (robot description, URDF)
Before this commit: robot sentient_static_upper_body, 36 links, 35 joints
Links:
- link camera_link: mass 0.264253 -> 0.264252
Joints:
- joint so101_camera_tilt_joint: origin xyz=-0.0202 -0.0188 -0.0234 rpy=1.5708 -5.24284e-08 3.14159265 -> xyz=0.0202 0.0188 -0.0234 rpy=1.5708 -5.24284e-08 -1.41553e-15
- joint zed2i_left_optical_joint: origin xyz=-0.05875235 -0.0149073367 0.0761937731 rpy=2.73522519 1.57079633 -0.948913556 -> xyz=0.0605510764 -0.00276305502 0.0761937731 rpy=-2.55382532 1.57079633 2.89272591

Commit message: ZED 2i: the camera frame is upright and the IMU's axes are the ones measured on the robot
allisa_bot's zed2i_left_optical_frame is the left eye of an upside-down camera: it sits on the
right lens with its x towards the robot's left. The composer turns the ZED frame half a turn
about its own x, so ZED_camera is upright and forward and the left eye lands on the left lens.

The ZED 2i's sensor module, as mounted, has x down, y towards the right eye and z out of the
back, not the axes read from zed-open-capture's README. Measured 2026-10-26 on the static upper
body: model and IMU agree at a new neck pose (pitch 12.7 vs 15.5 deg nose up, roll -3.2 vs
-1.6), and a +56 tick camera-tilt step (4.92 deg) moved the IMU 4.93 deg further nose up, the
sense the model gives the tilt joint.

Co-Authored-By: Claude Opus 5.5 <noreply@anthropic.com>

File: assets/sentient_static_upper_body/sentient_static_upper_body.urdf (robot description, URDF)
Before this commit: robot sentient_static_upper_body, 36 links, 35 joints
Joints:
- joint zed2i_left_optical_frame_to_ZED_camera: origin xyz=0.06 0 0 rpy=0.785398163 -1.57079633 0.785398163 -> xyz=0.06 0 0 rpy=-2.35619449 -1.57079633 0.785398163

Commit message: Static upper body: the camera tilt horn turns with the camera
allisa_bot exports the tilt servo horn into the fixed base_link at its CAD pose, so it hung in
the air beside the camera once the neck moved. It sits on the tilt axis (within 1 mm, face
square to it), so the composer moves it into camera_link at the place the source zero pose puts
it; it now stays on the tilt axis at every pose.

Co-Authored-By: Claude Opus 5.5 <noreply@anthropic.com>

File: assets/sentient_static_upper_body/sentient_static_upper_body.urdf (robot description, URDF)
Before this commit: robot sentient_static_upper_body, 36 links, 35 joints
Links:
- link base_link: mass 1.45907 -> 0.416388; geometry collision mesh filename=meshes/collision/base_link.stl; visual mesh filename=meshes/base_link.stl scale=1 1 1
- link camera_link: mass 0.264252 -> 0.264509; geometry collision mesh filename=meshes/collision/camera_link.stl; visual mesh filename=meshes/Camera_Component___Body___ZED_2i___4_6mm___Cover_ste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 scale=1 1 1

Commit message: Static upper body names the public SO-101 meshes instead of copying them
The static upper body vendored eight TheRobotStudio SO-101 STLs and an
Apache LICENSE under its proprietary folder. They were byte-identical to
assets/so101/meshes and assets/ai_worker/ffw_bg2_rev4/LICENSE, and the
asset store serves a shared digest under the stricter licence, so public
hosts were refused the public SO-101 meshes and the ai_worker licence.

The compose tool now names the neck meshes as
package://sx-embodiments/so101/meshes/..., the cross-package mechanism
aloha and the DAS gripper already use, and the copies are deleted.
Re-rendered the URDF, its digest, the asset manifest, driver bindings and
the render pack (pack.glb unchanged: same geometry). A new manifest test
refuses any public digest that is also entitled.

Co-Authored-By: Claude Opus 5.5 <noreply@anthropic.com>

File: assets/sentient_static_upper_body/sentient_static_upper_body.urdf (robot description, URDF)
Before this commit: robot sentient_static_upper_body, 36 links, 35 joints
Links:
- link so101_elbow_flex_link: geometry collision mesh filename=package://sx-embodiments/so101/meshes/motor_holder_so101_wr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; collision mesh filename=package://sx-embodiments/so101/meshes/sts3215_03a_v1.stl
- link so101_shoulder_lift_link: geometry collision mesh filename=package://sx-embodiments/so101/meshes/sts3215_03a_v1.stl; collision mesh filename=package://sx-embodiments/so101/meshes/upper_arm_so101_v1.stl
- link so101_shoulder_pan_link: geometry collision mesh filename=package://sx-embodiments/so101/meshes/motor_holder_so101_ba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; collision mesh filename=package://sx-embodiments/so101/meshes/rotation_pitch_so101_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
- link so101_wrist_flex_link: geometry collision mesh filename=package://sx-embodiments/so101/meshes/sts3215_03a_no_horn_v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; collision mesh filename=package://sx-embodiments/so101/meshes/wrist_roll_pitch_so10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
- link so101_wrist_roll_link: geometry collision mesh filename=meshes/Wrist_Roll_Follower_SO101_5__Fillet1.stl; collision mesh filename=package://sx-embodiments/so101/meshes/sts3215_03a_v1.stl

Commit message: Speeds as data: rated speeds in the registry, composed into the description; the derate is declared in commissioning
- ActuatorRating carries the vendor's rated output speed (DM4310 120 rpm, DM4340 36 rpm,
  DM8009 and DM-J8009P 100 rpm at 24 V, from their manuals), rendered into the drivers'
  vocabulary. compose_static_upper_body_urdf sets each Damiao joint's limit velocity from its
  bound model's rating instead of the CAD export's 0.5 rad/s placeholder (effort 54 stays: a
  follow-up). Re-rendered the URDF, its digest, the asset manifest, render pack, bindings and
  fixtures; the published revision is kept by digest for the historical document.
- tools/rekey_dynamics.py moves dynamics documents (docs/dynamics, the parity fixture, any
  bench calibration) to the new description only when the two differ in velocity limits alone;
  anything else is refused, to be identified again. Every document here is re-keyed.
- Commissioning declares a derate for this robot's over-rail axes ("derate": max_speed,
  max_acceleration; sx-commission --derate), replacing the automatic 0.3 rad/s and 1.5 rad/s^2
  for those axes with a person's recorded decision; the derate prints what it holds an axis to.

Co-Authored-By: Claude Opus 5.5 <noreply@anthropic.com>

File: assets/sentient_static_upper_body/sentient_static_upper_body.urdf (robot description, URDF)
Before this commit: robot sentient_static_upper_body, 36 links, 35 joints
Joints:
- joint left_elbow_pitch_joint: limit lower=-2.9753185320820936 upper=0.000953688868543523 effort=54 velocity=0.5 -> lower=-2.9753185320820936 upper=0.000953688868543523 effort=54 velocity=3.76991
- joint left_forearm_yaw_joint: limit lower=-6.82669565880827 upper=1.8839169909208824 effort=54 velocity=0.5 -> lower=-6.82669565880827 upper=1.8839169909208824 effort=54 velocity=3.76991
- joint left_shoulder_pitch_joint: limit lower=-2.642671854734111 upper=2.889868009460594 effort=54 velocity=0.5 -> lower=-2.642671854734111 upper=2.889868009460594 effort=54 velocity=10.472
- joint left_shoulder_roll_joint: limit lower=-0.3873884184023808 upper=1.2018387121385512 effort=54 velocity=0.5 -> lower=-0.3873884184023808 upper=1.2018387121385512 effort=54 velocity=10.472
- joint left_upper_arm_yaw_joint: limit lower=-5.1230258640421145 upper=0.8070115205615327 effort=54 velocity=0.5 -> lower=-5.1230258640421145 upper=0.8070115205615327 effort=54 velocity=3.76991
- joint left_wrist_pitch_joint: limit lower=-2.4408712901503016 upper=2.1280613412680243 effort=54 velocity=0.5 -> lower=-2.4408712901503016 upper=2.1280613412680243 effort=54 velocity=12.5664
- joint left_wrist_roll_joint: limit lower=-2.0967803463797967 upper=2.096017395284962 effort=54 velocity=0.5 -> lower=-2.0967803463797967 upper=2.096017395284962 effort=54 velocity=12.5664
- joint right_elbow_pitch_joint: limit lower=-0.029182879377431803 upper=2.966544594491493 effort=54 velocity=0.5 -> lower=-0.029182879377431803 upper=2.966544594491493 effort=54 velocity=3.76991
- joint right_forearm_yaw_joint: limit lower=-6.009575036240177 upper=1.4261463340199896 effort=54 velocity=0.5 -> lower=-6.009575036240177 upper=1.4261463340199896 effort=54 velocity=3.76991
- joint right_shoulder_pitch_joint: limit lower=-2.9139009689478907 upper=3.1225680933852136 effort=54 velocity=0.5 -> lower=-2.9139009689478907 upper=3.1225680933852136 effort=54 velocity=10.472
- joint right_shoulder_roll_joint: limit lower=-1.2101034267894413 upper=0.35464911018127765 effort=54 velocity=0.5 -> lower=-1.2101034267894413 upper=0.35464911018127765 effort=54 velocity=10.472
- joint right_upper_arm_yaw_joint: limit lower=-2.4210345616845963 upper=2.7597848477912574 effort=54 velocity=0.5 -> lower=-2.4210345616845963 upper=2.7597848477912574 effort=54 velocity=3.76991
- joint right_wrist_pitch_joint: limit lower=-2.255855649652858 upper=2.308880750743878 effort=54 velocity=0.5 -> lower=-2.255855649652858 upper=2.308880750743878 effort=54 velocity=12.5664
- joint right_wrist_roll_joint: limit lower=-2.0986877241168838 upper=2.112039368276493 effort=54 velocity=0.5 -> lower=-2.0986877241168838 upper=2.112039368276493 effort=54 velocity=12.5664
- joint torso_joint: limit lower=-1.221293965056839 upper=1.1499580376897836 effort=54 velocity=0.5 -> lower=-1.221293965056839 upper=1.1499580376897836 effort=54 velocity=10.472

Commit message: Speeds as data: refute findings; effort from the ratings; a declared derate records who decided it
- The description's effort is each Damiao joint's model peak torque too (the CAD export's
  54 N·m placeholder); one re-render and one re-key from the published description.
- A declared derate is a speed and the decision it records ("decided": who and why); its
  acceleration keeps the automatic ratio to speed, and no axis is derated faster than its
  model's rated speed. sx-commission --derate <rad/s>,<decided>, given once, and refused with
  --rail without the station it is recorded for.
- A derate reports the limits in force (the tighter of it and the governor's own).
- rekey_dynamics refuses a velocity or effort that is not a finite positive number, checks
  every document before writing any, and reports unreadable documents; tests cover a joint
  range change, and that every identified document names the current description.

Co-Authored-By: Claude Opus 5.5 <noreply@anthropic.com>

File: assets/sentient_static_upper_body/sentient_static_upper_body.urdf (robot description, URDF)
Before this commit: robot sentient_static_upper_body, 36 links, 35 joints
Joints:
- joint left_elbow_pitch_joint: limit lower=-2.9753185320820936 upper=0.000953688868543523 effort=54 velocity=3.76991 -> lower=-2.9753185320820936 upper=0.000953688868543523 effort=27 velocity=3.76991
- joint left_forearm_yaw_joint: limit lower=-6.82669565880827 upper=1.8839169909208824 effort=54 velocity=3.76991 -> lower=-6.82669565880827 upper=1.8839169909208824 effort=27 velocity=3.76991
- joint left_shoulder_pitch_joint: limit lower=-2.642671854734111 upper=2.889868009460594 effort=54 velocity=10.472 -> lower=-2.642671854734111 upper=2.889868009460594 effort=40 velocity=10.472
- joint left_shoulder_roll_joint: limit lower=-0.3873884184023808 upper=1.2018387121385512 effort=54 velocity=10.472 -> lower=-0.3873884184023808 upper=1.2018387121385512 effort=40 velocity=10.472
- joint left_upper_arm_yaw_joint: limit lower=-5.1230258640421145 upper=0.8070115205615327 effort=54 velocity=3.76991 -> lower=-5.1230258640421145 upper=0.8070115205615327 effort=27 velocity=3.76991
- joint left_wrist_pitch_joint: limit lower=-2.4408712901503016 upper=2.1280613412680243 effort=54 velocity=12.5664 -> lower=-2.4408712901503016 upper=2.1280613412680243 effort=7 velocity=12.5664
- joint left_wrist_roll_joint: limit lower=-2.0967803463797967 upper=2.096017395284962 effort=54 velocity=12.5664 -> lower=-2.0967803463797967 upper=2.096017395284962 effort=7 velocity=12.5664
- joint right_elbow_pitch_joint: limit lower=-0.029182879377431803 upper=2.966544594491493 effort=54 velocity=3.76991 -> lower=-0.029182879377431803 upper=2.966544594491493 effort=27 velocity=3.76991
- joint right_forearm_yaw_joint: limit lower=-6.009575036240177 upper=1.4261463340199896 effort=54 velocity=3.76991 -> lower=-6.009575036240177 upper=1.4261463340199896 effort=27 velocity=3.76991
- joint right_shoulder_pitch_joint: limit lower=-2.9139009689478907 upper=3.1225680933852136 effort=54 velocity=10.472 -> lower=-2.9139009689478907 upper=3.1225680933852136 effort=40 velocity=10.472
- joint right_shoulder_roll_joint: limit lower=-1.2101034267894413 upper=0.35464911018127765 effort=54 velocity=10.472 -> lower=-1.2101034267894413 upper=0.35464911018127765 effort=40 velocity=10.472
- joint right_upper_arm_yaw_joint: limit lower=-2.4210345616845963 upper=2.7597848477912574 effort=54 velocity=3.76991 -> lower=-2.4210345616845963 upper=2.7597848477912574 effort=27 velocity=3.76991
- joint right_wrist_pitch_joint: limit lower=-2.255855649652858 upper=2.308880750743878 effort=54 velocity=12.5664 -> lower=-2.255855649652858 upper=2.308880750743878 effort=7 velocity=12.5664
- joint right_wrist_roll_joint: limit lower=-2.0986877241168838 upper=2.112039368276493 effort=54 velocity=12.5664 -> lower=-2.0986877241168838 upper=2.112039368276493 effort=7 velocity=12.5664
- joint torso_joint: limit lower=-1.221293965056839 upper=1.1499580376897836 effort=54 velocity=10.472 -> lower=-1.221293965056839 upper=1.1499580376897836 effort=40 velocity=10.472
