Commit message: Static upper body: the head faces forward at the recalibrated neck zero
Owner at the robot, 10-27: the neck was recalibrated (camera tilt id 6: homing -575, range
1243..2745), and at its zero the ZED faces forward while the model had it 42 deg nose up
and the tilt reading outside the joint's range. CAMERA_RECALIBRATION (-0.734 rad) turns the
camera mount so the model's camera faces forward and level at the all-zero neck; the tilt
range (the free arc clear of the wrist) and home (now 0) turn with it. No capsule
self-collision at the neutral pose or anywhere in the new range.

The dynamics documents move to the new description: rekey_dynamics now also accepts a
re-render confined to links no identified joint carries (the neck's camera is on no arm),
and refuses one reaching an identified link or a joint a calibration or plan names.

Co-Authored-By: Claude Opus 5.5 <noreply@anthropic.com>

File: assets/sentient_static_upper_body/sentient_static_upper_body.urdf (robot description, URDF)
Before this commit: robot sentient_static_upper_body, 36 links, 35 joints
Joints:
- joint so101_camera_tilt_joint: limit lower=-3.14159265 upper=-0.261799388 effort=10 velocity=10 -> lower=-2.407592654 upper=0.472200612 effort=10 velocity=10
- joint zed2i_left_optical_joint: origin xyz=0.0605510764 -0.00276305502 0.0761937731 rpy=-2.55382532 1.57079633 2.89272591 -> xyz=0.0431084143 -0.0426114062 0.0761937731 rpy=-2.9378157 1.57079633 1.77473553

Commit message: Static upper body: the head mount fits the neck's measured forward rest
The 10-27 sample from the production room (neck at rest, ZED facing straight forward as
the owner saw it: pan -0.1926, lift -1.4730, elbow 1.7215, wrist flex -1.7392, roll
0.2417, tilt -1.0787 rad) replaces the all-zero assumption: CAMERA_RECALIBRATION -1.1476
puts the model's camera level and heading +0.01 deg there. Tilt range [-1.994, 0.886];
home tilt 0.4135, forward with the rest of the neck at zero. The description #158
published (ca769021) is kept beside a1589691 as a superseded revision the station
accepts fits against.

Co-Authored-By: Claude Opus 5.5 <noreply@anthropic.com>

File: assets/sentient_static_upper_body/sentient_static_upper_body.urdf (robot description, URDF)
Before this commit: robot sentient_static_upper_body, 36 links, 35 joints
Joints:
- joint so101_camera_tilt_joint: limit lower=-2.407592654 upper=0.472200612 effort=10 velocity=10 -> lower=-1.993966704 upper=0.885826562 effort=10 velocity=10
- joint zed2i_left_optical_joint: origin xyz=0.0431084143 -0.0426114062 0.0761937731 rpy=-2.9378157 1.57079633 1.77473553 -> xyz=0.0223461651 -0.0563446202 0.0761937731 rpy=2.85635293 1.57079633 0.872092909

Commit message: Static upper body: the neck's elbow and wrist flex reach its folded rest
The neck rests unpowered at elbow 1.7215 and wrist flex -1.7392 rad (measured 10-27),
past the official SO-101 limits (+-1.69, +-1.65806), against its servos' stops. The
limits are this build's calibrated reach rounded out (+-1.74, +-1.80); each unit's
calibration still bounds its servo. The previous description is kept as a superseded
revision the station accepts fits against.

Co-Authored-By: Claude Opus 5.5 <noreply@anthropic.com>

File: assets/sentient_static_upper_body/sentient_static_upper_body.urdf (robot description, URDF)
Before this commit: robot sentient_static_upper_body, 36 links, 35 joints
Joints:
- joint so101_elbow_flex_joint: limit lower=-1.69 upper=1.69 effort=10 velocity=10 -> lower=-1.74 upper=1.74 effort=10 velocity=10
- joint so101_wrist_flex_joint: limit lower=-1.65806 upper=1.65806 effort=10 velocity=10 -> lower=-1.80 upper=1.80 effort=10 velocity=10
