Commit message: Every described body draws: COLLADA colours, a collision fallback, one shape reader, StarArm's visuals
On top of #182 (COLLADA and capsules), render_pack.build now builds for every body whose
definition has a description:

- COLLADA meshes keep their materials' diffuse colours (a URDF material still wins), walk
  instance_node, take the first visual scene when a file names no scene, and turn X_UP
  files with the file's x up (it was mapped to +y). Node transforms are composed in plain
  floats and applied elementwise, so the bytes do not depend on the machine's BLAS. Each
  Franka and UR link matches its collision mesh's bounds within 2 percent.
- A description with no visual at all is drawn from its collision geometry, for every body.
- Visual and collision elements are read by one function (shapes) both modules use, and a
  mesh file is read once per process.
- StarArm102-LD's packaged URDF had its visuals stripped on import; it now keeps upstream's
  visual meshes at the same pinned revision (no collision, since the LD geometry is not
  qualified). The previous revision stays under _by_digest so recorded ids still resolve.

The committed packs and the tree-pose fixture are byte-identical.

insta360-umi is not drawn: its definition carries no description at all (its jaw is
unmeasured), so no registry consumer can materialize it. The new test pins it as the only
body left out and builds every other one within its declared budget, checking each link with
geometry has triangles.

Co-Authored-By: Claude Opus 5.5 <noreply@anthropic.com>

File: assets/stararm102/kinematics.urdf (robot description, URDF)
Before this commit: robot stararm102_description, 10 links, 9 joints
Links:
- link base_link: geometry visual mesh filename=package://sx-embodiments/stararm102/meshes/base_link.STL
- link link1: geometry visual mesh filename=package://sx-embodiments/stararm102/meshes/link1.STL
- link link2: geometry visual mesh filename=package://sx-embodiments/stararm102/meshes/link2.STL
- link link3: geometry visual mesh filename=package://sx-embodiments/stararm102/meshes/link3.STL
- link link4: geometry visual mesh filename=package://sx-embodiments/stararm102/meshes/link4.STL
- link link5: geometry visual mesh filename=package://sx-embodiments/stararm102/meshes/link5.STL
- link link6: geometry visual mesh filename=package://sx-embodiments/stararm102/meshes/link6.STL
- link link7_left: geometry visual mesh filename=package://sx-embodiments/stararm102/meshes/link7_left.STL
- link link7_right: geometry visual mesh filename=package://sx-embodiments/stararm102/meshes/link7_right.STL
